File: hw1.kicad_sch (KiCad schematic)
At the start: 18 parts, among them M1 Stepper_Motor, SW1 RotaryEncoder_Switch, SW2 SW_Back, SW5 SW_Bolus, SW6 SW_Settings, U4 XIAO-RP2350-DIP

Commit message: Added thicker traces for the whole MCU part. Still need to fix some DRC errors related to the XIAO's castellated pins.
Parts:
- renumbered SW5 to SW3, SW6 to SW4
Connections:
- net SW_BACK: now also U4.16 (GPIO20_D12_TX1); no longer U4.11 (GPIO3_D10_SPI0_MOSI)
- net SW_BOLUS: now also U4.11 (GPIO3_D10_SPI0_MOSI); no longer U4.16 (GPIO20_D12_TX1)
