File: power.kicad_sch (KiCad schematic)
At the start: 37 parts, among them J2 USB_C_Receptacle_USB2.0_16P, Q1 STL6P3LLH6, Q2 STL6P3LLH6, U2 STUSB4500QTR, U5 TPS54308DDCT

Commit message: Added LCSC codes, swapped extended components for basic ones, fixed labels and tidied schematics.
Parts:
- C50: LCSC C51205 -> C29823
- J2: LCSC C52209111 -> C2765186
- Q1, Q2: LCSC C457492 -> C49452349
- R1: LCSC C2907041 -> C23179
- R11, R5: LCSC C2907015 -> C31850
- R13: LCSC C2907089 -> C22775
- R2, R4: LCSC C2907440 -> C4410
- R3: LCSC C2906859 -> C25741
Changed lines of the file:
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@@
 			)
 		)
-		(property "LCSC" "C457492"
+		(property "LCSC" "C49452349"
 			(at 74.93 171.45 0)
 			(effects
@@
 			)
 		)
-		(property "LCSC" "C52209111"
+		(property "LCSC" "C2765186"
 			(at 156.21 44.45 0)
 			(effects
@@
 			)
 		)
-		(property "LCSC" "C2907041"
+		(property "LCSC" "C23179"
 			(at 127 135.89 0)
 			(effects
@@
 			)
 		)
-		(property "LCSC" "C2906859"
+		(property "LCSC" "C25741"
 			(at 99.06 44.45 0)
 			(effects
@@
 			)
 		)
-		(property "LCSC" "C2907015"
+		(property "LCSC" "C31850"
 			(at 44.45 184.15 0)
 			(effects
@@
 			)
 		)
-		(property "LCSC" "C51205"
+		(property "LCSC" "C29823"
 			(at 212.09 45.72 0)
 			(effects
@@
 			)
 		)
-		(property "LCSC" "C457492"
+		(property "LCSC" "C49452349"
 			(at 53.34 171.45 0)
 			(effects
@@
 			)
 		)
-		(property "LCSC" "C2907015"
+		(property "LCSC" "C31850"
 			(at 99.06 58.42 0)
 			(effects
@@
 			)
 		)
-		(property "LCSC" "C2907440"
+		(property "LCSC" "C4410"
 			(at 107.95 177.8 0)
 			(effects
@@
 			)
 		)
-		(property "LCSC" "C2907089"
+		(property "LCSC" "C22775"
 			(at 81.28 184.15 0)
 			(effects
@@
 			)
 		)
-		(property "LCSC" "C2907440"
+		(property "LCSC" "C4410"
 			(at 144.78 135.89 0)
 			(effects

Commit message: Finalised design, sent PCB to manufacturing
Connections:
- net SCL: now also JP5.1 (A); no longer JP6.1 (A)
- net SDA: now also JP6.1 (A); no longer JP5.1 (A)
Changed lines of the file:
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@@
 	(global_label "SDA"
 		(shape input)
-		(at 119.38 102.87 180)
+		(at 119.38 96.52 180)
 		(fields_autoplaced yes)
 		(effects
@@
 		)
 		(property "Intersheetrefs" "${INTERSHEET_REFS}"
-			(at 112.8267 102.87 0)
+			(at 112.8267 96.52 0)
 			(effects
 				(font
@@
 	(global_label "SCL"
 		(shape input)
-		(at 119.38 96.52 180)
+		(at 119.38 102.87 180)
 		(fields_autoplaced yes)
 		(effects
@@
 		)
 		(property "Intersheetrefs" "${INTERSHEET_REFS}"
-			(at 112.8872 96.52 0)
+			(at 112.8872 102.87 0)
 			(effects
 				(font
